File: eagle/igep-lcd.sch (EAGLE design)
At the start: 68 parts, among them IC1 LM1117IMPX-3.3, U1 SN74LVC8T245PW, U2 SN74LVC8T245PW, U3 SN74LVC8T245PW, U4 SN74LVC8T245PW

Commit message: First phase of PCD design
Connections:
- new net N$12: R5.1, U$7.TS2
- new net N$18: R3.1, U$7.TS1
- new net N$19: R10.1, U$4.EN
- new net N$24: R9.1, U$3.EN
- new net N$28: R8.1, U$2.EN
- new net N$3: R7.1, U$7.TS4
- new net N$30: C38.1, U3.B1
- new net N$32: C37.1, U3.B2
- new net N$37: C36.1, U3.B3
- new net N$38: C35.1, U3.B4
- new net N$39: C34.1, U3.B5
- new net N$40: C33.1, U3.B6
- new net N$41: C32.1, U3.B7
- new net N$42: C31.1, U3.B8
- new net N$43: C30.1, U2.B1
- new net N$44: C29.1, U2.B2
- new net N$45: C28.1, U2.B3
- new net N$46: C27.1, U2.B4
- new net N$47: C26.1, U2.B5
- new net N$48: C25.1, U2.B6
- new net N$49: C23.1, U2.B7
- new net N$50: C24.1, U2.B8
- new net N$51: C22.1, U1.B1
- new net N$52: C21.1, U1.B2
- new net N$53: C20.1, U1.B3
- new net N$54: C19.1, U1.B4
- new net N$55: C18.1, U1.B5
- new net N$56: C17.1, U1.B6
- new net N$57: C16.1, U1.B7
- new net N$58: C40.1, U1.B8
- new net N$6: R6.1, U$7.TS3
- net LCD_DATA0: no longer C22.1, U1.B1
- net LCD_DATA1: no longer C21.1, U1.B2
- net LCD_DATA10: no longer C28.1, U2.B3
- net LCD_DATA11: no longer C27.1, U2.B4
- net LCD_DATA12: no longer C26.1, U2.B5
- net LCD_DATA13: no longer C25.1, U2.B6
- net LCD_DATA14: no longer C23.1, U2.B7
- net LCD_DATA15: no longer C24.1, U2.B8
- net LCD_DATA16: no longer C38.1, U3.B1
- net LCD_DATA17: no longer C37.1, U3.B2
- net LCD_DATA18: no longer C36.1, U3.B3
- net LCD_DATA19: no longer C35.1, U3.B4
- net LCD_DATA2: no longer C20.1, U1.B3
- net LCD_DATA20: no longer C34.1, U3.B5
- net LCD_DATA21: no longer C33.1, U3.B6
- net LCD_DATA22: no longer C32.1, U3.B7
- net LCD_DATA23: no longer C31.1, U3.B8
- net LCD_DATA3: no longer C19.1, U1.B4
- net LCD_DATA4: no longer C18.1, U1.B5
- net LCD_DATA5: no longer C17.1, U1.B6
- net LCD_DATA6: no longer C16.1, U1.B7
- net LCD_DATA7: no longer C40.1, U1.B8
- net LCD_DATA8: no longer C30.1, U2.B1
- net LCD_DATA9: no longer C29.1, U2.B2
- net N$29: no longer R3.1, U$7.TS1
- net N$31: no longer R5.1, U$7.TS2
- net N$33: no longer R6.1, U$7.TS3
- net N$34: no longer R7.1, U$7.TS4
- net N$35: no longer R10.1, R8.1, R9.1, U$2.EN, U$3.EN, U$4.EN

Commit message: Updated schematics
Parts:
- added C12, C41, C42, C43: 100nF, rcl:C-EUC1206
Connections:
- net N$10: now also C42.1, C42.2
- net N$11: now also C43.1, C43.2
- net N$5: now also C41.1, C41.2
- net N$9: now also C12.1, C12.2
Changed lines of the file:
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@@
 <part name="R9" library="rcl" deviceset="R-EU_" device="R1206" value="0"/>
 <part name="R10" library="rcl" deviceset="R-EU_" device="R1206" value="0"/>
+<part name="C12" library="rcl" deviceset="C-EU" device="C1206" value="100nF"/>
+<part name="C41" library="rcl" deviceset="C-EU" device="C1206" value="100nF"/>
+<part name="C42" library="rcl" deviceset="C-EU" device="C1206" value="100nF"/>
+<part name="C43" library="rcl" deviceset="C-EU" device="C1206" value="100nF"/>
 </parts>
 <sheets>
@@
 <instance part="R9" gate="G$1" x="78.74" y="-226.06" rot="R90"/>
 <instance part="R10" gate="G$1" x="81.28" y="-287.02" rot="R90"/>
+<instance part="C12" gate="G$1" x="208.28" y="-68.58" rot="R90"/>
+<instance part="C41" gate="G$1" x="205.74" y="-66.04" rot="R90"/>
+<instance part="C42" gate="G$1" x="210.82" y="-71.12" rot="R90"/>
+<instance part="C43" gate="G$1" x="213.36" y="-73.66" rot="R90"/>
 </instances>
 <busses>
@@
 <segment>
 <pinref part="U4" gate="A" pin="B8"/>
-<wire x1="175.26" y1="-66.04" x2="312.42" y2="-66.04" width="0.1524" layer="91"/>
+<wire x1="175.26" y1="-66.04" x2="203.2" y2="-66.04" width="0.1524" layer="91"/>
+<wire x1="203.2" y1="-66.04" x2="210.82" y2="-66.04" width="0.1524" layer="91"/>
+<wire x1="210.82" y1="-66.04" x2="312.42" y2="-66.04" width="0.1524" layer="91"/>
 <wire x1="312.42" y1="-66.04" x2="312.42" y2="10.16" width="0.1524" layer="91"/>
 <pinref part="LCD" gate="-32" pin="1"/>
 <wire x1="312.42" y1="10.16" x2="320.04" y2="10.16" width="0.1524" layer="91"/>
+<pinref part="C41" gate="G$1" pin="1"/>
+<junction x="203.2" y="-66.04"/>
+<pinref part="C41" gate="G$1" pin="2"/>
+<junction x="210.82" y="-66.04"/>
 </segment>
 </net>
@@
 <wire x1="320.04" y1="7.62" x2="314.96" y2="7.62" width="0.1524" layer="91"/>
 <pinref part="U4" gate="A" pin="B7"/>
-<wire x1="175.26" y1="-68.58" x2="314.96" y2="-68.58" width="0.1524" layer="91"/>
+<wire x1="175.26" y1="-68.58" x2="205.74" y2="-68.58" width="0.1524" layer="91"/>
+<pinref part="C12" gate="G$1" pin="1"/>
+<wire x1="205.74" y1="-68.58" x2="213.36" y2="-68.58" width="0.1524" layer="91"/>
+<junction x="205.74" y="-68.58"/>
+<pinref part="C12" gate="G$1" pin="2"/>
+<wire x1="213.36" y1="-68.58" x2="314.96" y2="-68.58" width="0.1524" layer="91"/>
+<junction x="213.36" y="-68.58"/>
 </segment>
 </net>
@@
 <segment>
 <pinref part="U4" gate="A" pin="B6"/>
-<wire x1="175.26" y1="-71.12" x2="309.88" y2="-71.12" width="0.1524" layer="91"/>
+<wire x1="175.26" y1="-71.12" x2="208.28" y2="-71.12" width="0.1524" layer="91"/>
+<wire x1="208.28" y1="-71.12" x2="215.9" y2="-71.12" width="0.1524" layer="91"/>
+<wire x1="215.9" y1="-71.12" x2="309.88" y2="-71.12" width="0.1524" layer="91"/>
 <wire x1="309.88" y1="-71.12" x2="309.88" y2="15.24" width="0.1524" layer="91"/>
 <pinref part="LCD" gate="-30" pin="1"/>
 <wire x1="309.88" y1="15.24" x2="320.04" y2="15.24" width="0.1524" layer="91"/>
+<pinref part="C42" gate="G$1" pin="1"/>
+<junction x="208.28" y="-71.12"/>
+<pinref part="C42" gate="G$1" pin="2"/>
+<junction x="215.9" y="-71.12"/>
 </segment>
 </net>
@@
 <segment>
 <pinref part="U4" gate="A" pin="B5"/>
-<wire x1="175.26" y1="-73.66" x2="307.34" y2="-73.66" width="0.1524" layer="91"/>
+<wire x1="175.26" y1="-73.66" x2="210.82" y2="-73.66" width="0.1524" layer="91"/>
+<wire x1="210.82" y1="-73.66" x2="218.44" y2="-73.66" width="0.1524" layer="91"/>
+<wire x1="218.44" y1="-73.66" x2="307.34" y2="-73.66" width="0.1524" layer="91"/>
 <wire x1="307.34" y1="-73.66" x2="307.34" y2="5.08" width="0.1524" layer="91"/>
 <pinref part="LCD" gate="-34" pin="1"/>
 <wire x1="307.34" y1="5.08" x2="320.04" y2="5.08" width="0.1524" layer="91"/>
-</segment>
-</net>
+<pinref part="C43" gate="G$1" pin="1"/>
+<junction x="210.82" y="-73.66"/>
+<pinref part="C43" gate="G$1" pin="2"/>
+<junction x="218.44" y="-73.66"/>
+</segment>
+</net>

Commit message: Fixed postion testpads in schematic
Parts:
- added D11, D13, D7, D9: (no value), wirepad:1,6/0,8
Connections:
- net IGEP_LCD_DATA11: now also D11.P; no longer U$1.D11
- net IGEP_LCD_DATA13: now also D13.P; no longer U$1.D13
- net IGEP_LCD_DATA7: now also D7.P; no longer U$1.D7
- net IGEP_LCD_DATA9: now also D9.P; no longer U$1.D9
Changed lines of the file:
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@@
 <?xml version="1.0" encoding="utf-8"?>
 <!DOCTYPE eagle SYSTEM "eagle.dtd">
-<eagle version="6.1">
+<eagle version="6.2">
 <drawing>
 <settings>
@@
 <part name="C42" library="rcl" deviceset="C-EU" device="C1206" value="100nF"/>
 <part name="C43" library="rcl" deviceset="C-EU" device="C1206" value="100nF"/>
+<part name="D7" library="wirepad" deviceset="1,6/0,8" device=""/>
+<part name="D9" library="wirepad" deviceset="1,6/0,8" device=""/>
+<part name="D11" library="wirepad" deviceset="1,6/0,8" device=""/>
+<part name="D13" library="wirepad" deviceset="1,6/0,8" device=""/>
 </parts>
 <sheets>
@@
 <instance part="C42" gate="G$1" x="210.82" y="-71.12" rot="R90"/>
 <instance part="C43" gate="G$1" x="213.36" y="-73.66" rot="R90"/>
+<instance part="D7" gate="P" x="0" y="10.16" rot="R270"/>
+<instance part="D9" gate="P" x="7.62" y="10.16" rot="R270"/>
+<instance part="D11" gate="P" x="15.24" y="10.16" rot="R270"/>
+<instance part="D13" gate="P" x="22.86" y="10.16" rot="R270"/>
 </instances>
 <busses>
@@
 </segment>
 <segment>
-<pinref part="U$1" gate="G$1" pin="D7"/>
-<wire x1="43.18" y1="38.1" x2="38.1" y2="38.1" width="0.1524" layer="91"/>
+<pinref part="D7" gate="P" pin="P"/>
+<wire x1="0" y1="5.08" x2="0" y2="7.62" width="0.1524" layer="91"/>
 </segment>
 </net>
@@
 </segment>
 <segment>
-<pinref part="U$1" gate="G$1" pin="D9"/>
-<wire x1="43.18" y1="35.56" x2="38.1" y2="35.56" width="0.1524" layer="91"/>
+<pinref part="D9" gate="P" pin="P"/>
+<wire x1="7.62" y1="5.08" x2="7.62" y2="7.62" width="0.1524" layer="91"/>
 </segment>
 </net>
@@
 </segment>
 <segment>
-<pinref part="U$1" gate="G$1" pin="D11"/>
-<wire x1="43.18" y1="33.02" x2="38.1" y2="33.02" width="0.1524" layer="91"/>
+<pinref part="D11" gate="P" pin="P"/>
+<wire x1="15.24" y1="5.08" x2="15.24" y2="7.62" width="0.1524" layer="91"/>
 </segment>
 </net>
@@
 </segment>
 <segment>
-<pinref part="U$1" gate="G$1" pin="D13"/>
-<wire x1="43.18" y1="30.48" x2="38.1" y2="30.48" width="0.1524" layer="91"/>
-</segment>
-</net>
+<pinref part="D13" gate="P" pin="P"/>
+<wire x1="22.86" y1="5.08" x2="22.86" y2="7.62" width="0.1524" layer="91"/>
+</segment>
+</net>
